File: sensor_brd_2022.brd (EAGLE design)
At the start: 55 x 22 mm, 27 parts, among them J1 KMDGX-8S-BS, J2 SM06B-SRSS-TB__LF__SN_, J3 SM04B-SRSS-TB_LF__SN_, J4 1X4-BIG, U1 AD7730BR, U2 ADP3301ARZ-5, U3 24AA256-I_MF, Y1 4.9152MHz

Commit message: initial draft for layout
Parts:
- moved C9 1.94 mm to (6.10, 11.6)
- moved R1 1.66 mm to (27.8, 7.24)
- moved J1 1.02 mm to (50.5, 9.73)
- moved C7 0.92 mm to (39.8, 4.19)
- moved C10 0.90 mm to (15.6, 17.9)
- moved U2 0.64 mm to (34.9, 3.81)
- moved C5 0.64 mm to (15.6, 15.9)
- moved C1 0.25 mm to (30.2, 3.81)
- moved C6 0.25 mm to (27.7, 3.81)
Routing:
- net +5V: track 0.00 -> 52.7 mm, vias 0 -> 3
- net +5V/1: track 0.00 -> 39.2 mm
- net DGND: track 0.00 -> 30.7 mm, vias 0 -> 6
- net SCL: track 0.00 -> 28.5 mm, vias 0 -> 1
- net N$8: track 0.00 -> 25.2 mm, vias 0 -> 2
- net SDA: track 0.00 -> 23.7 mm, vias 0 -> 1
- net N$4: track 0.00 -> 23.4 mm, vias 0 -> 2
- net SCLK: track 0.00 -> 22.5 mm
- net E+: track 16.3 -> 38.0 mm, vias 0 -> 2
- net V+: track 0.00 -> 19.8 mm
- net E-: track 12.3 -> 31.9 mm
- net EN: track 0.00 -> 16.6 mm
- net AGND: track 0.00 -> 14.3 mm, vias 0 -> 5
- net DIN: track 0.00 -> 14.2 mm, vias 0 -> 1
- net N$6: track 0.00 -> 14.0 mm
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- added copper zone on layer 16, net AGND
- added copper zone on layer 16, net DGND

Commit message: First version send to JLCPCB
Parts:
- moved R5 8.78 mm to (37.2, 5.59)
- moved C1 8.51 mm to (30.5, 12.3)
- moved U2 8.51 mm to (35.2, 12.3)
- moved C7 8.26 mm to (39.6, 12.4)
- moved C6 7.24 mm to (27.8, 11.0)
- moved R1 7.24 mm to (27.8, 14.5)
- moved R7 6.75 mm to (37.2, 3.56)
- moved R8 6.75 mm to (37.2, 1.52)
- moved U3 6.75 mm to (30.9, 4.19)
- moved C11 6.41 mm to (32.0, 8.26)
- moved R4 4.73 mm to (37.2, 7.62)
- moved C10 0.13 mm to (15.6, 18.0)
Connections:
- net DGND: now also J1.2; no longer J1.8
- net DIN: now also J1.4; no longer J1.1
- net DOUT: now also J1.1; no longer J1.2
- net EN: now also J1.8; no longer J1.3
- net SCL: now also J1.6; no longer J1.5
- net SCLK: now also J1.7; no longer J1.4
- net SDA: now also J1.3; no longer J1.6
- net V+: now also J1.5; no longer J1.7
Routing:
- net N$8: track 25.2 -> 18.3 mm
- net SCL: track 28.5 -> 21.6 mm, vias 1 -> 0
- net N$4: track 23.4 -> 17.0 mm
- net V+: track 19.8 -> 14.5 mm
- net +5V: track 52.7 -> 57.7 mm, vias 3 -> 2
- net EN: track 16.6 -> 20.2 mm, vias 0 -> 1
- net DIN: track 14.2 -> 16.8 mm, vias 1 -> 0
- net SCLK: track 22.5 -> 20.1 mm
- net SDA: track 23.7 -> 21.8 mm
- net N$1: track 2.14 -> 4.04 mm
- net DOUT: track 12.8 -> 14.2 mm
- net DGND: track 30.7 -> 29.4 mm
- net +5V/1: track 39.2 -> 38.2 mm, vias 0 -> 2
